File: HW/audi_a4 door_indicator.kicad_sch (KiCad schematic)
At the start: 31 parts, among them CON1 15BrownLeftA_pin8, CON2 15BbrownRightA_pin7, CON3 15BlackRightA_pin13, CON4 15BlackRightA_pin12, CON5 10PurpleLeftA_pin5, SW1 DRIVER, SW2 PASSENGER, SW3 REAR LEFT, SW4 REAR RIGHT, SW5 TRUNK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

Commit message: updates
Parts:
- removed D? (x5): 1N4007, symbol diode:DIODE
- removed JP2: Jumper_NO_Small, symbol Device:Jumper_NO_Small
Connections:
- net GND: now also U1.28 ((SS)#D10), U1.4 (A0)
- net fis_data: no longer U1.22 (D4)
- new net radio_data: U1.22 (D4)

Commit message: new cable colours
Connections:
- net REAR_RIGHT renamed purple
- net purple: no longer D?.2 (K)
- net fis_clk renamed (cluster) grey
- net (cluster) grey: no longer U1.21 ((int3)#D3)
- net fis_data renamed (cluster) brown
- net fis_ena renamed (cluster) orange
- net (cluster) orange: no longer U1.20 ((int2)D2)
- net radio_data renamed (radio) brown
- new net  purple: D?.2 (K)
- new net (radio) grey: U1.21 ((int3)#D3)
- new net (radio) orange: U1.20 ((int2)D2)
Other:
- moved on the sheet: D?, U1
